File: cad/nano_m0.sch (KiCad schematic (older format))
At the start: 28 parts, among them J1 Conn_01x10, J2 Conn_01x10, J3 USB_B_Micro, J4 SWD, SW1 SW_SPST, SW2 SW_SPST, U1 AP2112K-3.3TRG1, U2 STM32F0706P6, Y1 16MHz

Commit message: changes to crystal
Parts:
- removed C3: 15pF, Capacitors_SMD:C_0805_HandSoldering, symbol device:C
- removed Y1: 16MHz, Crystals:Crystal_SMD_Abracon_ABM3B-4pin_5.0x3.2mm, symbol device:Crystal
- added X1: ASE-xxxMHz, Crystals:Crystal_SMD_Abracon_ABM3B-4pin_5.0x3.2mm, symbol Oscillators:ASE-xxxMHz
- C4: value 15pF -> .01uF
Connections:
- wire segments 131 -> 134
Changed lines of the file:
@@
 OSC_OUT
-$Comp
-L device:Crystal Y1
-U 1 1 5C0B9A41
-P 8450 5550
-F 0 "Y1" V 8404 5681 50  0000 L CNN
-F 1 "16MHz" V 8495 5681 50  0000 L CNN
-F 2 "Crystals:Crystal_SMD_Abracon_ABM3B-4pin_5.0x3.2mm" H 8450 5550 50  0001 C CNN
-F 3 "" H 8450 5550 50  0001 C CNN
-	1    8450 5550
-	0    1    1    0
-$EndComp
-$Comp
-L device:C C3
-U 1 1 5C0B9AAF
-P 7950 5400
-F 0 "C3" V 7698 5400 50  0000 C CNN
-F 1 "15pF" V 7789 5400 50  0000 C CNN
-F 2 "Capacitors_SMD:C_0805_HandSoldering" H 7988 5250 50  0001 C CNN
-F 3 "" H 7950 5400 50  0001 C CNN
-	1    7950 5400
-	0    1    1    0
-$EndComp
 $Comp
 L device:C C4
 U 1 1 5C0B9AFF
-P 7950 5700
-F 0 "C4" V 7698 5700 50  0000 C CNN
-F 1 "15pF" V 7789 5700 50  0000 C CNN
-F 2 "Capacitors_SMD:C_0805_HandSoldering" H 7988 5550 50  0001 C CNN
-F 3 "" H 7950 5700 50  0001 C CNN
-	1    7950 5700
-	0    1    1    0
+P 8050 5650
+F 0 "C4" V 7798 5650 50  0000 C CNN
+F 1 ".01uF" V 7889 5650 50  0000 C CNN
+F 2 "Capacitors_SMD:C_0805_HandSoldering" H 8088 5500 50  0001 C CNN
+F 3 "" H 8050 5650 50  0001 C CNN
+	1    8050 5650
+	-1   0    0    1
 $EndComp
 $Comp
 L power:GND #PWR0111
 U 1 1 5C0B9B4D
-P 7550 5900
-F 0 "#PWR0111" H 7550 5650 50  0001 C CNN
-F 1 "GND" H 7555 5727 50  0000 C CNN
-F 2 "" H 7550 5900 50  0001 C CNN
-F 3 "" H 7550 5900 50  0001 C CNN
-	1    7550 5900
-	1    0    0    -1
-$EndComp
-Wire Wire Line
-	7800 5400 7550 5400
-Wire Wire Line
-	7550 5400 7550 5700
-Wire Wire Line
-	7800 5700 7550 5700
-Connection ~ 7550 5700
-Wire Wire Line
-	7550 5700 7550 5900
-Wire Wire Line
-	8450 5400 8100 5400
-Wire Wire Line
-	8450 5700 8100 5700
-Wire Wire Line
-	8450 5400 9000 5400
-Connection ~ 8450 5400
-Wire Wire Line
-	8450 5700 9000 5700
-Connection ~ 8450 5700
-Text Label 8750 5400 0    50   ~ 0
-OSC_IN
-Text Label 8700 5700 0    50   ~ 0
-OSC_OUT
+P 8750 6100
+F 0 "#PWR0111" H 8750 5850 50  0001 C CNN
+F 1 "GND" H 8755 5927 50  0000 C CNN
+F 2 "" H 8750 6100 50  0001 C CNN
+F 3 "" H 8750 6100 50  0001 C CNN
+	1    8750 6100
+	1    0    0    -1
+$EndComp
 Wire Wire Line
 	9800 4050 10500 4050
@@
 Wire Notes Line
 	6700 600  6700 2300
-Text Notes 5850 750  0    50   ~ 0
+Text Notes 6450 750  0    50   ~ 0
 LEDs
 Wire Wire Line
@@
 Wire Notes Line
 	4400 2300 6700 2300
+$Comp
+L Oscillators:ASE-xxxMHz X1
+U 1 1 5C1A2FB8
+P 8750 5650
+F 0 "X1" H 9091 5696 50  0000 L CNN
+F 1 "ASE-xxxMHz" H 9091 5605 50  0000 L CNN
+F 2 "Crystals:Crystal_SMD_Abracon_ABM3B-4pin_5.0x3.2mm" H 9450 5300 50  0001 C CNN
+F 3 "http://www.abracon.com/Oscillators/ASV.pdf" H 8650 5650 50  0001 C CNN
+	1    8750 5650
+	1    0    0    -1
+$EndComp
+Wire Wire Line
+	8750 5350 8050 5350
+Wire Wire Line
+	8050 5350 8050 5500
+Wire Wire Line
+	8050 5800 8050 5950
+Wire Wire Line
+	8050 5950 8750 5950
+Wire Wire Line
+	8750 5950 8750 6100
+Connection ~ 8750 5950
+$Comp
+L power:+3.3V #PWR07
+U 1 1 5C1B9503
+P 8750 5100
+F 0 "#PWR07" H 8750 4950 50  0001 C CNN
+F 1 "+3.3V" H 8765 5273 50  0000 C CNN
+F 2 "" H 8750 5100 50  0001 C CNN
+F 3 "" H 8750 5100 50  0001 C CNN
+	1    8750 5100
+	1    0    0    -1
+$EndComp
+Wire Wire Line
+	8750 5100 8750 5150
+Connection ~ 8750 5350
+Wire Wire Line
+	8450 5650 8350 5650
+Wire Wire Line
+	8350 5650 8350 5150
+Wire Wire Line
+	8350 5150 8750 5150
+Connection ~ 8750 5150
+Wire Wire Line
+	8750 5150 8750 5350
+Wire Wire Line
+	9050 5650 9550 5650
+Text Label 9300 5650 0    50   ~ 0
+OSC_IN
 $EndSCHEMATC

Commit message: board v2
Parts:
- removed X1: ASE-xxxMHz, Crystals:Crystal_SMD_Abracon_ABM3B-4pin_5.0x3.2mm, symbol Oscillators:ASE-xxxMHz
- added C3: 22pF, Capacitors_SMD:C_0805_HandSoldering, symbol device:C
- added Y1: Crystal, Crystals:Crystal_SMD_SeikoEpson_TSX3225-4pin_3.2x2.5mm_HandSoldering, symbol device:Crystal
- C4: value .01uF -> 22pF
Connections:
- net labels removed: VBUS
- wire segments 134 -> 131
Changed lines of the file:
@@
 Text Label 7500 3650 0    50   ~ 0
 OSC_OUT
-$Comp
-L device:C C4
-U 1 1 5C0B9AFF
-P 8050 5650
-F 0 "C4" V 7798 5650 50  0000 C CNN
-F 1 ".01uF" V 7889 5650 50  0000 C CNN
-F 2 "Capacitors_SMD:C_0805_HandSoldering" H 8088 5500 50  0001 C CNN
-F 3 "" H 8050 5650 50  0001 C CNN
-	1    8050 5650
-	-1   0    0    1
-$EndComp
-$Comp
-L power:GND #PWR0111
-U 1 1 5C0B9B4D
-P 8750 6100
-F 0 "#PWR0111" H 8750 5850 50  0001 C CNN
-F 1 "GND" H 8755 5927 50  0000 C CNN
-F 2 "" H 8750 6100 50  0001 C CNN
-F 3 "" H 8750 6100 50  0001 C CNN
-	1    8750 6100
-	1    0    0    -1
-$EndComp
 Wire Wire Line
 	9800 4050 10500 4050
@@
 	4300 6800 4300 7100
 $Comp
-L power:VBUS #PWR0119
-U 1 1 5C0FFED2
-P 4100 900
-F 0 "#PWR0119" H 4100 750 50  0001 C CNN
-F 1 "VBUS" H 4115 1073 50  0000 C CNN
-F 2 "" H 4100 900 50  0001 C CNN
-F 3 "" H 4100 900 50  0001 C CNN
-	1    4100 900
-	1    0    0    -1
-$EndComp
-$Comp
-L power:VBUS #PWR0120
-U 1 1 5C0FFF4F
-P 3250 6100
-F 0 "#PWR0120" H 3250 5950 50  0001 C CNN
-F 1 "VBUS" H 3265 6273 50  0000 C CNN
-F 2 "" H 3250 6100 50  0001 C CNN
-F 3 "" H 3250 6100 50  0001 C CNN
-	1    3250 6100
-	1    0    0    -1
-$EndComp
-$Comp
 L device:Polyfuse F1
 U 1 1 5C102DC5
-P 3750 6400
-F 0 "F1" V 3525 6400 50  0000 C CNN
-F 1 "500mA" V 3616 6400 50  0000 C CNN
-F 2 "Fuse_Holders_and_Fuses:Fuse_SMD1206_HandSoldering" H 3800 6200 50  0001 L CNN
-F 3 "" H 3750 6400 50  0001 C CNN
-	1    3750 6400
+P 4150 6400
+F 0 "F1" V 3925 6400 50  0000 C CNN
+F 1 "500mA" V 4016 6400 50  0000 C CNN
+F 2 "Fuse_Holders_and_Fuses:Fuse_SMD1206_HandSoldering" H 4200 6200 50  0001 L CNN
+F 3 "" H 4150 6400 50  0001 C CNN
+	1    4150 6400
 	0    1    1    0
 $EndComp
-Wire Wire Line
-	4300 6400 3900 6400
-Connection ~ 4300 6400
-Wire Wire Line
-	3600 6400 3250 6400
-Wire Wire Line
-	3250 6400 3250 6100
 Wire Notes Line
 	11000 6350 11000 2800
@@
 Wire Wire Line
 	5650 3950 6100 3950
-Text Label 5950 5250 0    50   ~ 0
-BOOT
-Text Label 5950 5150 0    50   ~ 0
-NRST
 Text Label 5950 5050 0    50   ~ 0
 PA0
@@
 Text Label 5850 3550 0    50   ~ 0
 USB_N
-Wire Wire Line
-	4300 6400 4500 6400
-$Comp
-L power:+5V #PWR03
-U 1 1 5C1ACFC1
-P 4500 6050
-F 0 "#PWR03" H 4500 5900 50  0001 C CNN
-F 1 "+5V" H 4515 6223 50  0000 C CNN
-F 2 "" H 4500 6050 50  0001 C CNN
-F 3 "" H 4500 6050 50  0001 C CNN
-	1    4500 6050
-	1    0    0    -1
-$EndComp
 $Comp
 L power:+5V #PWR04
@@
 	0    1    1    0
 $EndComp
-Wire Wire Line
-	4500 6050 4500 6400
-Connection ~ 4500 6400
-Wire Wire Line
-	4500 6400 4650 6400
 $Comp
 L Connector:Conn_ARM_JTAG_SWD_10 J4
@@
 Wire Wire Line
 	3800 3700 3800 3500
-$Comp
-L power:+3.3V #PWR02
-U 1 1 5C0D1FE8
-P 3800 3500
-F 0 "#PWR02" H 3800 3350 50  0001 C CNN
-F 1 "+3.3V" H 3815 3673 50  0000 C CNN
-F 2 "" H 3800 3500 50  0001 C CNN
-F 3 "" H 3800 3500 50  0001 C CNN
-	1    3800 3500
-	1    0    0    -1
-$EndComp
 Wire Wire Line
 	4300 4000 4600 4000
@@
 Wire Notes Line
 	4400 2300 6700 2300
-$Comp
-L Oscillators:ASE-xxxMHz X1
-U 1 1 5C1A2FB8
-P 8750 5650
-F 0 "X1" H 9091 5696 50  0000 L CNN
-F 1 "ASE-xxxMHz" H 9091 5605 50  0000 L CNN
-F 2 "Crystals:Crystal_SMD_Abracon_ABM3B-4pin_5.0x3.2mm" H 9450 5300 50  0001 C CNN
-F 3 "http://www.abracon.com/Oscillators/ASV.pdf" H 8650 5650 50  0001 C CNN
-	1    8750 5650
-	1    0    0    -1
-$EndComp
-Wire Wire Line
-	8750 5350 8050 5350
-Wire Wire Line
-	8050 5350 8050 5500
-Wire Wire Line
-	8050 5800 8050 5950
-Wire Wire Line
-	8050 5950 8750 5950
-Wire Wire Line
-	8750 5950 8750 6100
-Connection ~ 8750 5950
-$Comp
-L power:+3.3V #PWR07
-U 1 1 5C1B9503
-P 8750 5100
-F 0 "#PWR07" H 8750 4950 50  0001 C CNN
-F 1 "+3.3V" H 8765 5273 50  0000 C CNN
-F 2 "" H 8750 5100 50  0001 C CNN
-F 3 "" H 8750 5100 50  0001 C CNN
-	1    8750 5100
-	1    0    0    -1
-$EndComp
-Wire Wire Line
-	8750 5100 8750 5150
-Connection ~ 8750 5350
-Wire Wire Line
-	8450 5650 8350 5650
-Wire Wire Line
-	8350 5650 8350 5150
-Wire Wire Line
-	8350 5150 8750 5150
-Connection ~ 8750 5150
-Wire Wire Line
-	8750 5150 8750 5350
-Wire Wire Line
-	9050 5650 9550 5650
-Text Label 9300 5650 0    50   ~ 0
+Wire Wire Line
+	4300 6400 4650 6400
+Connection ~ 4300 6400
+$Comp
+L power:+5V #PWR03
+U 1 1 5C21F9EA
+P 3750 6100
+F 0 "#PWR03" H 3750 5950 50  0001 C CNN
+F 1 "+5V" H 3765 6273 50  0000 C CNN
+F 2 "" H 3750 6100 50  0001 C CNN
+F 3 "" H 3750 6100 50  0001 C CNN
+	1    3750 6100
+	1    0    0    -1
+$EndComp
+Wire Wire Line
+	3750 6100 3750 6400
+Wire Wire Line
+	4000 6400 3750 6400
+$Comp
+L device:Crystal Y1
+U 1 1 5C2C7904
+P 8600 5450
+F 0 "Y1" H 8600 5718 50  0000 C CNN
+F 1 "Crystal" H 8600 5627 50  0000 C CNN
+F 2 "Crystals:Crystal_SMD_SeikoEpson_TSX3225-4pin_3.2x2.5mm_HandSoldering" H 8600 5450 50  0001 C CNN
+F 3 "" H 8600 5450 50  0001 C CNN
+	1    8600 5450
+	1    0    0    -1
+$EndComp
+$Comp
+L device:C C3
+U 1 1 5C2DD2F3
+P 8350 5750
+F 0 "C3" H 8465 5796 50  0000 L CNN
+F 1 "22pF" H 8465 5705 50  0000 L CNN
+F 2 "Capacitors_SMD:C_0805_HandSoldering" H 8388 5600 50  0001 C CNN
+F 3 "" H 8350 5750 50  0001 C CNN
+	1    8350 5750
+	1    0    0    -1
+$EndComp
+$Comp
+L device:C C4
+U 1 1 5C2DD35B
+P 8850 5750
+F 0 "C4" H 8965 5796 50  0000 L CNN
+F 1 "22pF" H 8965 5705 50  0000 L CNN
+F 2 "Capacitors_SMD:C_0805_HandSoldering" H 8888 5600 50  0001 C CNN
+F 3 "" H 8850 5750 50  0001 C CNN
+	1    8850 5750
+	1    0    0    -1
+$EndComp
+Wire Wire Line
+	8750 5450 8850 5450
+Wire Wire Line
+	8850 5450 8850 5600
+Wire Wire Line
+	8450 5450 8350 5450
+Wire Wire Line
+	8350 5450 8350 5600
+Wire Wire Line
+	8350 5450 8350 5000
+Connection ~ 8350 5450
+Wire Wire Line
+	8850 5450 8850 5000
+Connection ~ 8850 5450
+Text Label 8350 5000 0    50   ~ 0
 OSC_IN
+Text Label 8850 5000 0    50   ~ 0
+OSC_OUT
+$Comp
+L power:GND #PWR07
+U 1 1 5C2F3150
+P 8600 6050
+F 0 "#PWR07" H 8600 5800 50  0001 C CNN
+F 1 "GND" H 8605 5877 50  0000 C CNN
+F 2 "" H 8600 6050 50  0001 C CNN
+F 3 "" H 8600 6050 50  0001 C CNN
+	1    8600 6050
+	1    0    0    -1
+$EndComp
+Wire Wire Line
+	8850 5900 8850 6000
+Wire Wire Line
+	8850 6000 8600 6000
+Wire Wire Line
+	8600 6000 8600 6050
+Wire Wire Line
+	8350 5900 8350 6000
+Wire Wire Line
+	8350 6000 8600 6000
+Connection ~ 8600 6000
+$Comp
+L power:+5V #PWR0111
+U 1 1 5C304EC4
+P 4100 900
+F 0 "#PWR0111" H 4100 750 50  0001 C CNN
+F 1 "+5V" H 4115 1073 50  0000 C CNN
+F 2 "" H 4100 900 50  0001 C CNN
+F 3 "" H 4100 900 50  0001 C CNN
+	1    4100 900
+	1    0    0    -1
+$EndComp
+$Comp
+L power:+3.3V #PWR0119
+U 1 1 5C3052E4
+P 3800 3500
+F 0 "#PWR0119" H 3800 3350 50  0001 C CNN
+F 1 "+3.3V" H 3815 3673 50  0000 C CNN
+F 2 "" H 3800 3500 50  0001 C CNN
+F 3 "" H 3800 3500 50  0001 C CNN
+	1    3800 3500
+	1    0    0    -1
+$EndComp
+Text Label 5950 5150 0    50   ~ 0
+BOOT
+Text Label 5950 5250 0    50   ~ 0
+NRST
 $EndSCHEMATC

Commit message: final v3 board
Parts:
- removed JP1: Jumper_NC_Small, Jumper:SolderJumper-2_P1.3mm_Bridged_Pad1.0x1.5mm, symbol device:Jumper_NC_Small
- removed JP2: Jumper_NO_Small, Jumper:SolderJumper-2_P1.3mm_Open_Pad1.0x1.5mm, symbol device:Jumper_NO_Small
- C1, C2, C3, C4, C5, C6, C7: footprint Capacitors_SMD:C_0805_HandSoldering -> Capacitors_SMD:C_0805
- D1, D2, D3: footprint LEDs:LED_0805_HandSoldering -> LEDs:LED_0805
- R1, R2, R5: value 80ohm -> 100; footprint Resistors_SMD:R_0805_HandSoldering -> Resistors_SMD:R_0805
- R3, R4, R6: footprint Resistors_SMD:R_0805_HandSoldering -> Resistors_SMD:R_0805
- Y1: footprint Crystals:Crystal_SMD_SeikoEpson_TSX3225-4pin_3.2x2.5mm_HandSoldering -> Crystals:Crystal_SMD_SeikoEpson_TSX3225-4pin_3.2x2.5mm
Connections:
- wire segments 131 -> 126
Other:
- note added: "External Button"
- moved on the sheet: SW1

Commit message: update schematic symbols to kicad5
Parts:
- C1, C2, C3, C4, C5, C6, C7: symbol device:C -> nano_m0-rescue:C-device
- D1, D2, D3: symbol device:LED -> nano_m0-rescue:LED-device
- F1: symbol device:Polyfuse -> nano_m0-rescue:Polyfuse-device
- J1, J2: symbol Connector:Conn_01x10 -> nano_m0-rescue:Conn_01x10-Connector
- R1, R2, R3, R4, R5, R6: symbol device:R -> nano_m0-rescue:R-device
- Y1: symbol device:Crystal -> nano_m0-rescue:Crystal-device
Changed lines of the file:
@@
 $EndComp
 $Comp
-L device:R R3
+L nano_m0-rescue:R-device R3
 U 1 1 5C0B5007
 P 7750 1750
@@
 	9800 1450 10100 1450
 $Comp
-L device:R R4
+L nano_m0-rescue:R-device R4
 U 1 1 5C0B57F1
 P 10100 1200
@@
 $EndComp
 $Comp
-L device:C C7
+L nano_m0-rescue:C-device C7
 U 1 1 5C0B5846
 P 10350 1700
@@
 $EndComp
 $Comp
-L device:C C6
+L nano_m0-rescue:C-device C6
 U 1 1 5C0B7322
 P 10300 5550
@@
 $EndComp
 $Comp
-L device:C C5
+L nano_m0-rescue:C-device C5
 U 1 1 5C0B7397
 P 9900 5550
@@
 PA1
 $Comp
-L device:LED D1
+L nano_m0-rescue:LED-device D1
 U 1 1 5C0C1A5D
 P 4600 1300
@@
 $EndComp
 $Comp
-L device:R R1
+L nano_m0-rescue:R-device R1
 U 1 1 5C0C1B92
 P 4600 1750
@@
 $EndComp
 $Comp
-L device:C C2
+L nano_m0-rescue:C-device C2
 U 1 1 5C0EEF05
 P 6300 6650
@@
 Connection ~ 4650 6400
 $Comp
-L device:C C1
+L nano_m0-rescue:C-device C1
 U 1 1 5C0FA4CC
 P 4300 6650
@@
 	4300 6800 4300 7100
 $Comp
-L device:Polyfuse F1
+L nano_m0-rescue:Polyfuse-device F1
 U 1 1 5C102DC5
 P 4150 6400
@@
 PA13
 $Comp
-L Connector:Conn_01x10 J2
+L nano_m0-rescue:Conn_01x10-Connector J2
 U 1 1 5C16ACC6
 P 5450 5050
@@
 $EndComp
 $Comp
-L Connector:Conn_01x10 J1
+L nano_m0-rescue:Conn_01x10-Connector J1
 U 1 1 5C16AD71
 P 5450 3650
@@
 $EndComp
 $Comp
-L device:R R2
+L nano_m0-rescue:R-device R2
 U 1 1 5C0C7FC9
 P 5350 1750
@@
 $EndComp
 $Comp
-L device:LED D2
+L nano_m0-rescue:LED-device D2
 U 1 1 5C0C7FC2
 P 5350 1300
@@
 $EndComp
 $Comp
-L device:R R5
+L nano_m0-rescue:R-device R5
 U 1 1 5C0DF2B9
 P 6100 1750
@@
 $EndComp
 $Comp
-L device:LED D3
+L nano_m0-rescue:LED-device D3
 U 1 1 5C0DF2C0
 P 6100 1300
@@
 	6100 1900 6100 2050
 $Comp
-L device:R R6
+L nano_m0-rescue:R-device R6
 U 1 1 5C0F1F04
 P 8300 1400
@@
 	4000 6400 3750 6400
 $Comp
-L device:Crystal Y1
+L nano_m0-rescue:Crystal-device Y1
 U 1 1 5C2C7904
 P 8600 5450
@@
 $EndComp
 $Comp
-L device:C C3
+L nano_m0-rescue:C-device C3
 U 1 1 5C2DD2F3
 P 8350 5750
@@
 $EndComp
 $Comp
-L device:C C4
+L nano_m0-rescue:C-device C4
 U 1 1 5C2DD35B
 P 8850 5750
